Commit message: Change joint names to pan and tilt

File: urdf/dynamixel_pan_tilt.urdf.xacro (robot description, xacro)
@@ -35,5 +35,5 @@
   </link>
   <!-- Joint 1 -->
-  <joint name="joint1" type="revolute">
+  <joint name="pan" type="revolute">
     <parent link="link1"/>
     <child link="link2"/>
@@ -66,5 +66,5 @@
   </link>
   <!--  Joint 2 -->
-  <joint name="joint2" type="revolute">
+  <joint name="tilt" type="revolute">
     <parent link="link2"/>
     <child link="cam_base"/>

Commit message: Change to black material

File: urdf/dynamixel_pan_tilt.urdf.xacro (robot description, xacro)
@@ -2,7 +2,4 @@
 <!-- Open_Manipulator Chain -->
 <robot xmlns:xacro="http://ros.org/wiki/xacro" name="dynamixel_pan_tilt">
-  <material name="grey">
-    <color rgba="0.5 0.5 0.5 1.0"/>
-  </material>
   <!--  Joint 0 -->
   <joint name="camera_mount_to_dynamixel_pan_tilt" type="fixed">
@@ -18,5 +15,5 @@
         <mesh filename="package://open_manipulator_description/meshes/chain_link1.stl" scale="0.001 0.001 0.001"/>
       </geometry>
-      <material name="grey"/>
+      <material name="black"/>
     </visual>
     <collision>
@@ -49,5 +46,5 @@
         <mesh filename="package://open_manipulator_description/meshes/chain_link2.stl" scale="0.001 0.001 0.001"/>
       </geometry>
-      <material name="grey"/>
+      <material name="black"/>
     </visual>
     <collision>
@@ -68,9 +65,30 @@
   <joint name="tilt" type="revolute">
     <parent link="link2"/>
-    <child link="cam_base"/>
+    <child link="link3"/>
     <origin xyz="0.0 0.0 0.0595" rpy="0 0 0"/>
     <axis xyz="0 1 0"/>
     <limit velocity="4.8" effort="1" lower="${-pi*0.57}" upper="${pi*0.5}" />
   </joint>
-   <link name="cam_base"/>
+   <link name="link3">
+    <visual>
+      <origin xyz="0 0 0" rpy="0 0 1.5708"/>
+      <geometry>
+        <mesh filename="package://dynamixel_pan_tilt/meshes/link_3.stl" scale="1 1 1"/>
+      </geometry>
+      <material name="black"/>
+    </visual>
+    <collision>
+      <origin xyz="0 0 0" rpy="0 0 1.5708"/>
+      <geometry>
+        <mesh filename="package://dynamixel_pan_tilt/meshes/link_3.stl" scale="1 1 1"/>
+      </geometry>
+    </collision>
+    <inertial>
+      <origin xyz="-3.0184870e-04 5.4043684e-04 ${0.018 + 2.9433464e-02}" />
+      <mass value="9.8406837e-02" />
+      <inertia ixx="3.4543422e-05" ixy="-1.6031095e-08" ixz="-3.8375155e-07"
+               iyy="3.2689329e-05" iyz="2.8511935e-08"
+               izz="1.8850320e-05" />
+    </inertial>
+   </link>
 </robot>

Commit message: Add offset between link3 and camera_base

File: urdf/dynamixel_pan_tilt.urdf.xacro (robot description, xacro)
@@ -92,3 +92,10 @@
     </inertial>
    </link>
+  <link name="camera_base"/>
+    <!--  Joint 2 -->
+  <joint name="camera_base" type="fixed">
+    <parent link="link3"/>
+    <child link="camera_base"/>
+    <origin xyz="0.0 0.0 0.04" rpy="0 0 0"/>
+  </joint>
 </robot>

Commit message: corrected distance to top of pan-tilt

File: urdf/dynamixel_pan_tilt.urdf.xacro (robot description, xacro)
@@ -97,5 +97,5 @@
     <parent link="link3"/>
     <child link="camera_base"/>
-    <origin xyz="0.0 0.0 0.04" rpy="0 0 0"/>
+    <origin xyz="0.0 0.0 0.027" rpy="0 0 0"/>
   </joint>
 </robot>
